Commit message: Updated robot_core

File: description/robot_core.xacro (robot description, xacro)
@@ -1,4 +1,31 @@
 <?xml version="1.0"?>
-<robot xmlns:xacro="http://www.ros.org/wiki/xacro"  name="robot">
-    <xacro:include filename="robot_core.xacro">
+<robot xmlns:xacro="http://www.ros.org/wiki/xacro">
+    <material name="white">
+        <color rgba = "1 1 1 1 " />
+    </material>
+    <material name="orange">
+        <color rgba = "1 0.3 0.1 1 " />
+    </material>
+    <material name="blue">
+        <color rgba = "0.2 0.2 1 1 " />
+    </material>
+    <material name="black">
+        <color rgba = "0 0 0 1 " />
+    </material>
+    <link name = "base_link">
+    </link>
+    <joint name = "chassis_joint" type = "fixed">
+        <parent link = "base_link"/>
+        <child LINK = "chassis"/>
+        <origin xyz ="-0.1 0 0 "/>
+    </joint>
+    <link name = "chassis">
+        <visual>
+            <origin xyz = "0.15 0 0.075"/>
+            <geometry>
+                <box size = "0.3 0.3 0.15"/>
+            </geometry>
+            <material name = "white"/>
+        </visual>
+    <link/>
 </robot>

Commit message: changed robot core

File: description/robot_core.xacro (robot description, xacro)
@@ -1,22 +1,22 @@
 <?xml version="1.0"?>
 <robot xmlns:xacro="http://www.ros.org/wiki/xacro">
-    <material name="white">
-        <color rgba = "1 1 1 1 " />
+    <material name = "white">
+        <color rgba = "1 1 1 1"/>
     </material>
-    <material name="orange">
-        <color rgba = "1 0.3 0.1 1 " />
+    <material name = "orange">
+        <color rgba = "1 0.3 0.1 1"/>
     </material>
-    <material name="blue">
-        <color rgba = "0.2 0.2 1 1 " />
+    <material name = "blue">
+        <color rgba = "0.2 0.2 1 1"/>
     </material>
-    <material name="black">
-        <color rgba = "0 0 0 1 " />
+    <material name = "black">
+        <color rgba = "0 0 0 1"/>
     </material>
     <link name = "base_link">
     </link>
-    <joint name = "chassis_joint" type = "fixed">
+    <joint name = "chassis_joint" type="fixed">
         <parent link = "base_link"/>
-        <child LINK = "chassis"/>
-        <origin xyz ="-0.1 0 0 "/>
+        <child link = "chassis"/>
+        <origin xyz = "-0.1 0 0"/>
     </joint>
     <link name = "chassis">
@@ -24,8 +24,7 @@
             <origin xyz = "0.15 0 0.075"/>
             <geometry>
-                <box size = "0.3 0.3 0.15"/>
+                <box box size "0.3 0.3 0.15"/>
             </geometry>
-            <material name = "white"/>
         </visual>
-    <link/>
+    </link>
 </robot>

Commit message: update

File: description/robot_core.xacro (robot description, xacro)
@@ -24,5 +24,5 @@
             <origin xyz = "0.15 0 0.075"/>
             <geometry>
-                <box box size "0.3 0.3 0.15"/>
+                <box size= "0.3 0.3 0.15"/>
             </geometry>
         </visual>

Commit message: added wheels

File: description/robot_core.xacro (robot description, xacro)
@@ -13,6 +13,8 @@
         <color rgba = "0 0 0 1"/>
     </material>
+<!-- BASE LINK -->
     <link name = "base_link">
     </link>
+<!-- CHASSIS LINK -->
     <joint name = "chassis_joint" type="fixed">
         <parent link = "base_link"/>
@@ -28,3 +30,33 @@
         </visual>
     </link>
+<!-- LEFT WHEEL LINK -->
+    <joint name ="left_wheel_joint" type = "continuous">
+        <parent link = "base_link"/>
+        <child link = "left wheel"/>
+        <origin xyz = "0 0.175 0" rpy="-$(pi/2) 0 0"/>
+        <axis xyz = "0 0 1"/>
+    </joint>
+    <link name = "left_wheel">
+        <visual>
+            <geometry>
+                <cylinder radius = "0.05" length = "0.04"/>
+            </geometry>
+            <material name = "blue"/>
+        </visual>
+    </link>
+<!-- RIGHT WHEEL LINK -->
+    <joint name ="right_wheel_joint" type = "continuous">
+        <parent link = "base_link"/>
+        <child link = "left wheel"/>
+        <origin xyz = "0 -0.175 0" rpy="$(pi/2) 0 0"/>
+        <axis xyz = "0 0 -1"/>
+    </joint>
+    <link name = "right_wheel">
+        <visual>
+            <geometry>
+                <cylinder radius = "0.05" length = "0.04"/>
+            </geometry>
+            <material name = "blue"/>
+        </visual>
+    </link>
 </robot>

Commit message: fixed errors in wheels

File: description/robot_core.xacro (robot description, xacro)
@@ -33,5 +33,5 @@
     <joint name ="left_wheel_joint" type = "continuous">
         <parent link = "base_link"/>
-        <child link = "left wheel"/>
+        <child link = "left_wheel"/>
         <origin xyz = "0 0.175 0" rpy="-$(pi/2) 0 0"/>
         <axis xyz = "0 0 1"/>
@@ -48,5 +48,5 @@
     <joint name ="right_wheel_joint" type = "continuous">
         <parent link = "base_link"/>
-        <child link = "left wheel"/>
+        <child link = "right_wheel"/>
         <origin xyz = "0 -0.175 0" rpy="$(pi/2) 0 0"/>
         <axis xyz = "0 0 -1"/>

Commit message: fixed wheels pt.2

File: description/robot_core.xacro (robot description, xacro)
@@ -49,5 +49,5 @@
         <parent link = "base_link"/>
         <child link = "right_wheel"/>
-        <origin xyz = "0 -0.175 0" rpy="$(pi/2) 0 0"/>
+        <origin xyz = "0 -0.175 0" rpy="${pi/2} 0 0"/>
         <axis xyz = "0 0 -1"/>
     </joint>

Commit message: fix wheel pt.3

File: description/robot_core.xacro (robot description, xacro)
@@ -34,5 +34,5 @@
         <parent link = "base_link"/>
         <child link = "left_wheel"/>
-        <origin xyz = "0 0.175 0" rpy="-$(pi/2) 0 0"/>
+        <origin xyz = "0 0.175 0" rpy="-${pi/2} 0 0"/>
         <axis xyz = "0 0 1"/>
     </joint>

Commit message: caster wheel added

File: description/robot_core.xacro (robot description, xacro)
@@ -60,3 +60,17 @@
         </visual>
     </link>
+<!-- CASTER WHEEL LINK-->
+    <joint name ="caster_wheel_joint" type="fixed">
+        <parent link = "chassis"/>
+        <child link = "caster"/>
+        <origin xyz = "0.24 0 0"/>
+    </joint>
+    <link name ="caster_wheel">
+        <visual>
+            <geometry>
+                <sphere radius = "0.05"/>
+            </geometry>
+            <material name = "black"/>
+        </visual>
+    </link>
 </robot>

Commit message: fixed caster wheel

File: description/robot_core.xacro (robot description, xacro)
@@ -63,5 +63,5 @@
     <joint name ="caster_wheel_joint" type="fixed">
         <parent link = "chassis"/>
-        <child link = "caster"/>
+        <child link = "caster_wheel"/>
         <origin xyz = "0.24 0 0"/>
     </joint>

Commit message: created collisions

File: description/robot_core.xacro (robot description, xacro)
@@ -28,5 +28,12 @@
                 <box size= "0.3 0.3 0.15"/>
             </geometry>
+            <material name="white"/>
         </visual>
+        <collision>
+            <origin xyz = "0.15 0 0.075"/>
+            <geometry>
+                <box size= "0.3 0.3 0.15"/>
+            </geometry>
+        </collision>
     </link>
 <!-- LEFT WHEEL LINK -->
@@ -44,4 +51,9 @@
             <material name = "blue"/>
         </visual>
+        <collision>
+            <geometry>
+                <cylinder radius = "0.05" length = "0.04"/>
+            </geometry>
+        </collision>
     </link>
 <!-- RIGHT WHEEL LINK -->
@@ -59,4 +71,9 @@
             <material name = "blue"/>
         </visual>
+        <collision>
+            <geometry>
+                <cylinder radius = "0.05" length = "0.04"/>
+            </geometry>
+        </collision>
     </link>
 <!-- CASTER WHEEL LINK-->
@@ -73,4 +90,9 @@
             <material name = "black"/>
         </visual>
+        <collision>
+            <geometry>
+                <sphere radius = "0.05"/>
+            </geometry>
+        </collision>
     </link>
 </robot>

Commit message: inertia tagged

File: description/robot_core.xacro (robot description, xacro)
@@ -1,4 +1,5 @@
 <?xml version="1.0"?>
 <robot xmlns:xacro="http://www.ros.org/wiki/xacro">
+    <xacro: include filename="inertial_macros.xacro"/>
     <material name = "white">
         <color rgba = "1 1 1 1"/>
@@ -36,4 +37,7 @@
             </geometry>
         </collision>
+        <xacro:inertial_box mass="0.5" x="0.3" y="0.3" z="0.15">
+            <origin xyz ="0.15 0 0.075" rpy = "0 0 0"/>
+        </xacro:inertial_box>
     </link>
 <!-- LEFT WHEEL LINK -->
@@ -56,4 +60,7 @@
             </geometry>
         </collision>
+        <xacro:inertial_cylinder mass = "0.1" length ="0.04" radius = "0.05">
+            <origin xyz = "0 0 0" rpy = " 0 0 0"/>
+        </xacro:inertial_cylinder>
     </link>
 <!-- RIGHT WHEEL LINK -->
@@ -76,4 +83,7 @@
             </geometry>
         </collision>
+        <xacro:inertial_cylinder mass = "0.1" length ="0.04" radius = "0.05">
+            <origin xyz = "0 0 0" rpy = " 0 0 0"/>
+        </xacro:inertial_cylinder>
     </link>
 <!-- CASTER WHEEL LINK-->
@@ -95,4 +105,7 @@
             </geometry>
         </collision>
+        <xacro:inertial_cylinder mass="0.1" radius="0.05">
+            <origin xyz="0 0 0" rpy="0 0 0"/>
+        </xacro:inertial_cylinder>
     </link>
 </robot>
